Commit message: from omin retarget dataset

File: src/holosoma_retargeting/holosoma_retargeting/models/g1/g1_29dof.urdf (robot description, URDF)
Before this commit: robot g1_29dof, 55 links, 54 joints
Links:
- removed link left_pinky_link
- removed link left_thumb_link
- removed link right_pinky_link
- removed link right_thumb_link
- link right_ankle_roll_link: geometry collision mesh filename=assets/right_ankle_roll_link.obj; collision sphere radius=0.005
Joints:
- removed joint left_pinky_joint
- removed joint left_thumb_joint
- removed joint right_pinky_joint
- removed joint right_thumb_joint

File: src/holosoma_retargeting/holosoma_retargeting/models/g1/g1_29dof_spherehand.urdf (robot description, URDF)
Before this commit: robot g1_29dof, 53 links, 52 joints
Links:
- link right_ankle_roll_link: geometry collision mesh filename=assets/right_ankle_roll_link.obj; collision sphere radius=0.005
